File: pcb/dream_controller.kicad_pcb (KiCad board)
At the start: 2 copper layers, 17.8 x 45.7 mm, 4 parts, among them J1 Touchplate, J2 Joystick, U1 Teensy-LC, U2 MCP4922

Commit message: Complete schematic
Parts:
- moved U2 1.02 mm to (139.7, 124.5)
- moved J2 0.89 mm to (137.7, 128.9)
Routing:
- net +3V3: track 0.00 -> 47.0 mm, vias 0 -> 2
- net /CAP_CS: track 19.9 -> 10.3 mm
- net GND: track 0.00 -> 6.91 mm, vias 0 -> 26
- net /CAP_DR: track 17.0 -> 23.9 mm, vias 2 -> 0
- net /DAC_LATCH: track 31.6 -> 32.6 mm
- net /DAC_DATA: track 40.9 -> 41.9 mm
- net /CAP_CLK: track 16.7 -> 17.3 mm, vias 3 -> 1
- net /DAC_CLK: track 25.1 -> 25.7 mm, vias 2 -> 1
- net /CAP_COPI: track 9.43 -> 9.18 mm, vias 0 -> 1
Other:
- outline, holes or cut-outs redrawn
- board text added: "VREF"
- board text added: "X"
- board text added: "Y"

Commit message: Cleanup
Routing:
- net GND: track 6.91 -> 9.14 mm
- net /CAP_DR: track 23.9 -> 22.3 mm
Other:
- board text added: "JLCJLCJLCJLC"
Changed lines of the file:
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@@
     (effects (font (size 1 1) (thickness 0.15)) (justify mirror))
+  )
+  (gr_text "JLCJLCJLCJLC" (at 134.62 91.44) (layer "F.SilkS")
+    (effects (font (size 0.5 0.5) (thickness 0.1)))
   )
   (segment (start 141.515499 126.41) (end 142.5625 126.41) (width 0.25) (layer "F.Cu") (net 1))
@@
   (segment (start 138.43 95.25) (end 142.24 91.44) (width 0.25) (layer "B.Cu") (net 1))
   (segment (start 127 87.122) (end 129.286 89.408) (width 0.25) (layer "F.Cu") (net 2))
+  (segment (start 132.806 123.226) (end 132.806 124.7875) (width 0.25) (layer "F.Cu") (net 2))
   (segment (start 142.5625 125.11) (end 141.240113 125.11) (width 0.25) (layer "F.Cu") (net 2))
   (segment (start 127 86.36) (end 127 87.122) (width 0.25) (layer "F.Cu") (net 2))
   (segment (start 136.8375 125.11) (end 137.81 125.11) (width 0.25) (layer "F.Cu") (net 2))
   (segment (start 141.240113 125.11) (end 141.170107 125.039994) (width 0.25) (layer "F.Cu") (net 2))
+  (segment (start 132.806 124.7875) (end 132.334 125.2595) (width 0.25) (layer "F.Cu") (net 2))
   (segment (start 137.81 125.11) (end 138.176 125.476) (width 0.25) (layer "F.Cu") (net 2))
   (via (at 138.176 125.476) (size 0.8) (drill 0.4) (layers "F.Cu" "B.Cu") (net 2))
@@
   (via (at 139.7 87.63) (size 0.8) (drill 0.4) (layers "F.Cu" "B.Cu") (free) (net 2))
   (via (at 133.35 97.79) (size 0.8) (drill 0.4) (layers "F.Cu" "B.Cu") (free) (net 2))
-  (via (at 135.255 129.54) (size 0.8) (drill 0.4) (layers "F.Cu" "B.Cu") (free) (net 2))
   (via (at 136.525 100.965) (size 0.8) (drill 0.4) (layers "F.Cu" "B.Cu") (free) (net 2))
   (via (at 140.335 95.25) (size 0.8) (drill 0.4) (layers "F.Cu" "B.Cu") (free) (net 2))
+  (via (at 128.524 125.476) (size 0.8) (drill 0.4) (layers "F.Cu" "B.Cu") (free) (net 2))
   (via (at 134.62 114.3) (size 0.8) (drill 0.4) (layers "F.Cu" "B.Cu") (free) (net 2))
   (via (at 132.08 111.76) (size 0.8) (drill 0.4) (layers "F.Cu" "B.Cu") (free) (net 2))
@@
   (via (at 140.335 97.79) (size 0.8) (drill 0.4) (layers "F.Cu" "B.Cu") (free) (net 2))
   (via (at 132.08 106.68) (size 0.8) (drill 0.4) (layers "F.Cu" "B.Cu") (free) (net 2))
+  (via (at 132.334 125.2595) (size 0.8) (drill 0.4) (layers "F.Cu" "B.Cu") (net 2))
   (via (at 141.170107 125.039994) (size 0.8) (drill 0.4) (layers "F.Cu" "B.Cu") (net 2))
   (via (at 140.335 100.33) (size 0.8) (drill 0.4) (layers "F.Cu" "B.Cu") (free) (net 2))
   (via (at 129.286 89.408) (size 0.8) (drill 0.4) (layers "F.Cu" "B.Cu") (net 2))
   (via (at 134.62 104.14) (size 0.8) (drill 0.4) (layers "F.Cu" "B.Cu") (free) (net 2))
-  (via (at 127.635 129.54) (size 0.8) (drill 0.4) (layers "F.Cu" "B.Cu") (free) (net 2))
   (via (at 135.255 118.11) (size 0.8) (drill 0.4) (layers "F.Cu" "B.Cu") (free) (net 2))
   (segment (start 129.806 116.852) (end 129.794 116.84) (width 0.25) (layer "F.Cu") (net 8))
@@
   (via (at 129.794 116.84) (size 0.8) (drill 0.4) (layers "F.Cu" "B.Cu") (net 8))
   (segment (start 129.794 116.84) (end 127 116.84) (width 0.25) (layer "B.Cu") (net 8))
-  (segment (start 129.306 125.964) (end 129.306 127.726) (width 0.25) (layer "F.Cu") (net 9))
-  (segment (start 129.54 125.73) (end 129.306 125.964) (width 0.25) (layer "F.Cu") (net 9))
+  (segment (start 129.794 125.984) (end 129.306 126.472) (width 0.25) (layer "F.Cu") (net 9))
+  (segment (start 132.842 125.984) (end 129.794 125.984) (width 0.25) (layer "F.Cu") (net 9))
+  (segment (start 129.306 127.726) (end 129.306 126.472) (width 0.25) (layer "F.Cu") (net 9))
+  (segment (start 133.606489 125.219511) (end 132.842 125.984) (width 0.25) (layer "F.Cu") (net 9))
   (segment (start 127 111.76) (end 133.606489 118.366489) (width 0.25) (layer "F.Cu") (net 9))
-  (segment (start 129.306 127.726) (end 129.306 126.004) (width 0.25) (layer "F.Cu") (net 9))
-  (segment (start 133.606489 124.524533) (end 132.401022 125.73) (width 0.25) (layer "F.Cu") (net 9))
-  (segment (start 132.401022 125.73) (end 129.54 125.73) (width 0.25) (layer "F.Cu") (net 9))
-  (segment (start 133.606489 118.366489) (end 133.606489 124.524533) (width 0.25) (layer "F.Cu") (net 9))
+  (segment (start 133.606489 118.366489) (end 133.606489 125.219511) (width 0.25) (layer "F.Cu") (net 9))
   (segment (start 128.831 115.115) (end 128.778 115.062) (width 0.25) (layer "F.Cu") (net 10))
   (segment (start 128.831 123.226) (end 128.831 115.115) (width 0.25) (layer "F.Cu") (net 10))
@@
   (zone (net 0) (net_name "") (layer "F.Cu") (hatch edge 0.508)
     (connect_pads (clearance 0))
+    (min_thickness 0.254)
+    (keepout (tracks allowed) (vias allowed) (pads allowed ) (copperpour not_allowed) (footprints allowed))
+    (fill (thermal_gap 0.508) (thermal_bridge_width 0.508))
+    (polygon
+      (pts
+        (xy 140.97 128.016)
+        (xy 140.716 128.27)
+        (xy 139.446 128.016)
+        (xy 137.922 126.492)
+        (xy 137.922 125.73)
+        (xy 138.684 125.476)
+      )
+    )
+  )
+  (zone (net 0) (net_name "") (layer "F.Cu") (hatch edge 0.508)
+    (connect_pads (clearance 0))

Commit message: Additional cleanup
Routing:
- net /CAP_CS: track 10.3 -> 9.68 mm, vias 1 -> 0
- net GND: vias 26 -> 25
Changed lines of the file:
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@@
     (property "Sheetname" "")
     (attr smd)
-    (fp_text reference "U2" (at 0 0) (layer "F.SilkS")
+    (fp_text reference "U2" (at 0 0) (layer "F.SilkS") hide
       (effects (font (size 1 1) (thickness 0.15)))
     )
@@
   (via (at 136.525 100.965) (size 0.8) (drill 0.4) (layers "F.Cu" "B.Cu") (free) (net 2))
   (via (at 140.335 95.25) (size 0.8) (drill 0.4) (layers "F.Cu" "B.Cu") (free) (net 2))
-  (via (at 128.524 125.476) (size 0.8) (drill 0.4) (layers "F.Cu" "B.Cu") (free) (net 2))
   (via (at 134.62 114.3) (size 0.8) (drill 0.4) (layers "F.Cu" "B.Cu") (free) (net 2))
   (via (at 132.08 111.76) (size 0.8) (drill 0.4) (layers "F.Cu" "B.Cu") (free) (net 2))
@@
   (segment (start 127 111.76) (end 133.606489 118.366489) (width 0.25) (layer "F.Cu") (net 9))
   (segment (start 133.606489 118.366489) (end 133.606489 125.219511) (width 0.25) (layer "F.Cu") (net 9))
-  (segment (start 128.831 115.115) (end 128.778 115.062) (width 0.25) (layer "F.Cu") (net 10))
-  (segment (start 128.831 123.226) (end 128.831 115.115) (width 0.25) (layer "F.Cu") (net 10))
-  (via (at 128.778 115.062) (size 0.8) (drill 0.4) (layers "F.Cu" "B.Cu") (net 10))
-  (segment (start 127.762 115.062) (end 127 114.3) (width 0.25) (layer "B.Cu") (net 10))
-  (segment (start 128.778 115.062) (end 127.762 115.062) (width 0.25) (layer "B.Cu") (net 10))
+  (segment (start 128.831 123.226) (end 128.831 116.131) (width 0.25) (layer "F.Cu") (net 10))
+  (segment (start 128.831 116.131) (end 127 114.3) (width 0.25) (layer "F.Cu") (net 10))
   (segment (start 128.331 126.807) (end 127 125.476) (width 0.25) (layer "F.Cu") (net 11))
   (segment (start 128.331 127.726) (end 128.331 126.807) (width 0.25) (layer "F.Cu") (net 11))
@@
       )
     )
+  )
+  (zone (net 0) (net_name "") (layer "F.Cu") (hatch edge 0.508)
+    (connect_pads (clearance 0))
+    (min_thickness 0.254)
+    (keepout (tracks allowed) (vias allowed) (pads allowed ) (copperpour not_allowed) (footprints allowed))
+    (fill (thermal_gap 0.508) (thermal_bridge_width 0.508))
+    (polygon
+      (pts
+        (xy 133.096 125.984)
+        (xy 127.508 125.984)
+        (xy 127.508 124.968)
+        (xy 133.096 124.968)
+      )
+    )
+  )
+  (zone (net 0) (net_name "") (layer "F.Cu") (hatch edge 0.508)
+    (connect_pads (clearance 0))
+    (min_thickness 0.254)
+    (keepout (tracks allowed) (vias allowed) (pads not_allowed ) (copperpour not_allowed) (footprints allowed))
+    (fill (thermal_gap 0.508) (thermal_bridge_width 0.508))
+    (polygon
+      (pts
+        (xy 136.398 122.936)
+        (xy 134.112 122.936)
+        (xy 134.112 121.412)
+        (xy 136.398 121.412)
+      )
+    )

Commit message: silkscreen name
Other:
- board text added: "eric halin march 2022 dream-controller v.01"
Changed lines of the file:
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@@
     (pad_to_mask_clearance 0)
     (pcbplotparams
-      (layerselection 0x00010fc_ffffffff)
+      (layerselection 0x00010f0_ffffffff)
       (disableapertmacros false)
       (usegerberextensions false)
       (usegerberattributes true)
       (usegerberadvancedattributes true)
-      (creategerberjobfile true)
+      (creategerberjobfile false)
       (svguseinch false)
       (svgprecision 6)
@@
       (outputformat 1)
       (mirror false)
-      (drillshape 1)
+      (drillshape 0)
       (scaleselection 1)
-      (outputdirectory "")
+      (outputdirectory "export/")
     )
   )
@@
     (effects (font (size 1 1) (thickness 0.15)) (justify mirror))
   )
+  (gr_text "eric halin march 2022\ndream-controller v.01" (at 135.382 103.378 90) (layer "B.SilkS")
+    (effects (font (size 0.8 0.8) (thickness 0.15)) (justify mirror))
+  )
   (gr_text "JLCJLCJLCJLC" (at 134.62 91.44) (layer "F.SilkS")
